Commit message: Debugged

File: description/lidar.xacro (robot description, xacro)
@@ -2,8 +2,8 @@
 <robot xmlns:xacro="http://www.ros.org/wiki/xacro">
     <joint name="laser_joint" type="fixed">
-        <parent link="chassis"/>
+        <parent link="lid"/>
         <child link="laser_frame"/>
         <!-- Change origin in a minute -->
-        <origin xyz="0 0 0.36" rpy="0 0 0"/>
+        <origin xyz="-0.09525 0 0.04" rpy="0 0 3.1415"/>
     </joint>
     <link name="laser_frame">

File: description/robot.urdf.xacro (robot description, xacro)
@@ -12,4 +12,4 @@
     <xacro:include filename="lidar.xacro" />
     <xacro:include filename="camera.xacro" />
-    <xacro:include filename="face.xacro" />
+    <!-- <xacro:include filename="rear_camera.xacro" /> -->
 </robot>

File: description/robot_core.xacro (robot description, xacro)
@@ -16,4 +16,9 @@
     <xacro:property name="caster_wheel_offset_x" value="0.075"/>
     <xacro:property name="caster_wheel_offset_z" value="${wheel_offset_z - wheel_radius + caster_wheel_radius}"/>
+    <xacro:property name="chassis_top_length" value="0.4064"/>
+    <xacro:property name="chassis_top_width" value="0.254"/>
+    <xacro:property name="chassis_top_height" value="0.1905"/>
+    <xacro:property name="chassis_top_mass" value="0.0"/>
+    <xacro:property name="lid_thickness" value="0.0254"/>
     <material name="white">
         <color rgba="1 1 1 1" />
@@ -60,5 +65,5 @@
                 <box size="${chassis_length} ${chassis_width} ${chassis_height}"/>
             </geometry>
-            <material name="gold"/>
+            <material name="black"/>
         </visual>
         <collision>
@@ -73,5 +78,53 @@
     </link>
     <gazebo reference="chassis">
+        <material>Gazebo/Black</material>
+    </gazebo>
+    <!-- CHASSIS TOP LINK -->
+    <joint name="chassis_top_joint" type="fixed">
+        <origin xyz="${chassis_length/2} 0 ${chassis_height}" rpy="0 0 0" />
+        <parent link="chassis"/>
+        <child link="chassis_top"/>
+    </joint>
+    <link name="chassis_top">
+        <visual>
+            <origin xyz="0 0 ${chassis_top_height/2}"/>
+            <geometry>
+                <box size="${chassis_top_length} ${chassis_top_width} ${chassis_top_height}" />
+            </geometry>
+            <material name="gold" />
+        </visual>
+        <collision>
+            <origin xyz="0 0 0" rpy="0 0 0" />
+            <geometry>
+                <box size="${chassis_top_length} ${chassis_top_width} ${chassis_top_height}" />
+            </geometry>
+        </collision>
+    </link>
+    <gazebo reference="chassis_top">
         <material>Gazebo/Gold</material>
+    </gazebo>
+    <!-- LID LINK -->
+    <joint name="lid_joint" type="fixed">
+        <origin xyz="0 0 ${chassis_top_height}" />
+        <parent link="chassis_top"/>
+        <child link="lid"/>
+    </joint>
+    <link name="lid">
+        <visual>
+            <origin xyz="0 0 ${lid_thickness/2}" />
+            <geometry>
+                <box size="${chassis_top_length} ${chassis_top_width} ${lid_thickness}" />
+            </geometry>
+            <material name="black" />
+        </visual>
+        <collision>
+            <origin xyz="0 0 ${lid_thickness}" />
+            <geometry>
+                <box size="${chassis_top_length} ${chassis_top_width} ${lid_thickness}" />
+            </geometry>
+        </collision>
+    </link>
+    <gazebo reference="lid">
+        <material>Gazebo/Black</material>
     </gazebo>
     <!-- LEFT WHEEL LINK -->

File: description/ros2_control.xacro (robot description, xacro)
@@ -8,8 +8,8 @@
                 <param name="right_wheel_name">right_wheel_joint</param>
                 <param name="loop_rate">30</param>
-                <param name="device">/dev/ttyUSB0</param>
+                <param name="device">/dev/ttyACM0</param>
                 <param name="baud_rate">57600</param>
                 <param name="timeout">1000</param>
-                <param name="enc_counts_per_rev">3436</param>
+                <param name="enc_counts_per_rev">2525</param>
             </hardware>
             <joint name="left_wheel_joint">
